File: PCB/PCB/PCB.kicad_pcb (KiCad board)
At the start: 2 copper layers, 92.2 x 69.5 mm, 14 parts, among them J1 Alimentación, J2 AlimSensor1, J3 AlimSensor2, J4 AlimSensor1, J5 SensorArduino, J6 AlimSensor2, J7 CircuitoPotencia, SW1 SW_MEC_5G

Commit message: Actualización PCB
Routing:
- net GND: track 231.8 -> 260.9 mm, vias 2 -> 1
- net Net-(J6-Pin_1): track 34.9 -> 38.8 mm
- net Net-(J4-Pin_2): track 15.5 -> 12.8 mm
- net Net-(J4-Pin_1): track 15.3 -> 12.8 mm
- net Net-(J1-Pin_2): track 81.4 -> 81.1 mm, vias 2 -> 1
Other:
- board text removed: "Arduino"
- board text removed: "Power"
- board text removed: "S1Pow"
- board text removed: "S2Pow"
- board text removed: "Sig"
- board text removed: "SignalOut"
