File: Prototipo/PCB/PCB/_autosave-PCB.kicad_sch (KiCad schematic)
At the start: 16 parts, among them J1 Alimentación, J2 AlimSensor1, J3 AlimSensor2, J4 AlimSensor1, J5 SensorArduino, J6 AlimSensor2, J7 CircuitoPotencia, SW1 SW_MEC_5G, SW2 Interruptor

Commit message: suuuuu
Parts:
- removed R6: R, symbol Device:R
- removed SW2: Interruptor, Button_Switch_THT:Button2P, symbol Switch:SW_MEC_5G
Changed lines of the file:
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@@
   (junction (at 87.63 71.12) (diameter 0) (color 0 0 0 0)
   )
-  (junction (at 148.59 90.17) (diameter 0) (color 0 0 0 0)
-  )
   (junction (at 86.36 26.67) (diameter 0) (color 0 0 0 0)
   )
@@
     (stroke (width 0) (type default))
   )
-  (wire (pts (xy 148.59 90.17) (xy 148.59 91.44))
-    (stroke (width 0) (type default))
-  )
   (wire (pts (xy 179.07 30.48) (xy 179.07 26.67))
     (stroke (width 0) (type default))
@@
     (stroke (width 0) (type default))
   )
-  (wire (pts (xy 148.59 87.63) (xy 148.59 90.17))
-    (stroke (width 0) (type default))
-  )
   (wire (pts (xy 64.77 26.67) (xy 86.36 26.67))
     (stroke (width 0) (type default))
@@
     (stroke (width 0) (type default))
   )
-  (wire (pts (xy 148.59 90.17) (xy 154.94 90.17))
-    (stroke (width 0) (type default))
-  )
   (wire (pts (xy 113.03 34.29) (xy 113.03 26.67))
     (stroke (width 0) (type default))
@@
   (wire (pts (xy 114.3 52.07) (xy 114.3 58.42))
     (stroke (width 0) (type default))
-  )
-  (global_label "Pin arduino" (shape input) (at 154.94 90.17 0) (fields_autoplaced)
-    (effects (font (size 1.27 1.27)) (justify left))
-    (property "Intersheetrefs" "${INTERSHEET_REFS}" (at 169.0526 90.17 0)
-      (effects (font (size 1.27 1.27)) (justify left) hide)
-    )
   )
   (symbol (lib_id "Device:R") (at 114.3 62.23 0) (unit 1)
@@
     )
   )
-  (symbol (lib_id "power:GND") (at 148.59 101.6 0) (unit 1)
-    (in_bom yes) (on_board yes) (dnp no) (fields_autoplaced)
-    (property "Reference" "#PWR09" (at 148.59 107.95 0)
-      (effects (font (size 1.27 1.27)) hide)
-    )
-    (property "Value" "GND" (at 148.59 106.68 0)
-      (effects (font (size 1.27 1.27)))
-    )
-    (property "Footprint" "" (at 148.59 101.6 0)
-      (effects (font (size 1.27 1.27)) hide)
-    )
-    (property "Datasheet" "" (at 148.59 101.6 0)
-      (effects (font (size 1.27 1.27)) hide)
-    )
-    (pin "1")
-    (instances
-      (project "PCB"
-        (path "/2e02e944-af2e-473e-addd-61049117dc53"
-          (reference "#PWR09") (unit 1)
-        )
-      )
-    )
-  )
   (symbol (lib_id "power:GND") (at 162.56 38.1 0) (unit 1)
     (in_bom yes) (on_board yes) (dnp no) (fields_autoplaced)
@@
         (path "/2e02e944-af2e-473e-addd-61049117dc53"
           (reference "#PWR04") (unit 1)
-        )
-      )
-    )
-  )
-  (symbol (lib_id "Device:R") (at 148.59 83.82 0) (unit 1)
-    (in_bom yes) (on_board yes) (dnp no)
-    (property "Reference" "R6" (at 151.13 82.55 0)
-      (effects (font (size 1.27 1.27)) (justify left) hide)
-    )
-    (property "Value" "R" (at 151.13 83.82 0)
-      (effects (font (size 1.27 1.27)) (justify left))
-    )
-    (property "Footprint" "" (at 146.812 83.82 90)
-      (effects (font (size 1.27 1.27)) hide)
-    )
-    (property "Datasheet" "~" (at 148.59 83.82 0)
-      (effects (font (size 1.27 1.27)) hide)
-    )
-    (pin "1")
-    (pin "2")
-    (instances
-      (project "PCB"
-        (path "/2e02e944-af2e-473e-addd-61049117dc53"
-          (reference "R6") (unit 1)
         )
       )
@@
     )
   )
-  (symbol (lib_id "Switch:SW_MEC_5G") (at 148.59 96.52 270) (unit 1)
-    (in_bom yes) (on_board yes) (dnp no)
-    (property "Reference" "SW2" (at 152.4 95.25 90)
-      (effects (font (size 1.27 1.27)) (justify left) hide)
-    )
-    (property "Value" "Interruptor" (at 152.4 96.52 90)
-      (effects (font (size 1.27 1.27)) (justify left))
-    )
-    (property "Footprint" "Button_Switch_THT:Button2P" (at 153.67 96.52 0)
-      (effects (font (size 1.27 1.27)) hide)
-    )
-    (property "Datasheet" "http://www.apem.com/int/index.php?controller=attachment&id_attachment=488" (at 153.67 96.52 0)
-      (effects (font (size 1.27 1.27)) hide)
-    )
-    (pin "1")
-    (pin "3")
-    (pin "2")
-    (pin "4")
-    (instances
-      (project "PCB"
-        (path "/2e02e944-af2e-473e-addd-61049117dc53"
-          (reference "SW2") (unit 1)
-        )
-      )
-    )
-  )
   (symbol (lib_id "Device:R") (at 147.32 43.18 0) (unit 1)
     (in_bom yes) (on_board yes) (dnp no) (fields_autoplaced)
@@
         )
       )
-    )
-  )
-  (symbol (lib_id "power:+15V") (at 148.59 80.01 0) (unit 1)
-    (in_bom yes) (on_board yes) (dnp no) (fields_autoplaced)
-    (property "Reference" "#PWR08" (at 148.59 83.82 0)
-      (effects (font (size 1.27 1.27)) hide)
-    )
-    (property "Value" "+15V" (at 148.59 74.93 0)
-      (effects (font (size 1.27 1.27)))
-    )
-    (property "Footprint" "" (at 148.59 80.01 0)
-      (effects (font (size 1.27 1.27)) hide)
-    )
-    (property "Datasheet" "" (at 148.59 80.01 0)
-      (effects (font (size 1.27 1.27)) hide)
-    )
-    (pin "1")
-    (instances
-      (project "PCB"
-        (path "/2e02e944-af2e-473e-addd-61049117dc53"
-          (reference "#PWR08") (unit 1)
-        )
-      )
