File: Prototipo/PCB/PCB/PCB.kicad_sch (KiCad schematic)
At the start: 14 parts, among them J1 Alimentación, J2 AlimSensor1, J3 AlimSensor2, J4 AlimSensor1, J5 SensorArduino, J6 AlimSensor2, J7 CircuitoPotencia, SW1 SW_MEC_5G

Commit message: Big push
Cambio en la distribución
Prototipo terminado
Parts:
- J1: value Alimentación -> Alimentación 15V
- J4: value AlimSensor1 -> Señales
- J5: value SensorArduino -> Señal Arduino
- J6: value AlimSensor2 -> Control Rele
- J7: value CircuitoPotencia -> Alimentacion Solenoide
- SW1: value SW_MEC_5G -> Interruptor
- renumbered U3 to PRMA
Other:
- moved on the sheet: J4, J5, J6, J7, PRMA, R1, R2, R3, R4, R5, SW1
